Commit message: gripper gazebo

File: inspire_description/urdf/inspire_gripper.urdf.xacro (robot description, xacro)
@@ -16,5 +16,5 @@
                 <origin xyz="0 0 0" rpy="0 0 0" />
                 <geometry>
-                    <mesh filename="package://inspire_description/meshes/camera_connect.STL" />
+                    <mesh filename="file://$(find inspire_description)/meshes/camera_connect.STL" />
                 </geometry>
                 <material name="">
@@ -25,5 +25,5 @@
                 <origin xyz="0 0 0" rpy="0 0 0" />
                 <geometry>
-                    <mesh filename="package://inspire_description/meshes/camera_connect.STL" />
+                    <mesh filename="file://$(find inspire_description)/meshes/camera_connect.STL" />
                 </geometry>
             </collision>
@@ -44,5 +44,5 @@
                 <origin xyz="0 0 0" rpy="0 0 0" />
                 <geometry>
-                    <mesh filename="package://inspire_description/meshes/gripper_base_link.STL" />
+                    <mesh filename="file://$(find inspire_description)/meshes/gripper_base_link.STL" />
                 </geometry>
                 <material name="">
@@ -53,5 +53,5 @@
                 <origin xyz="0 0 0" rpy="0 0 0" />
                 <geometry>
-                    <mesh filename="package://inspire_description/meshes/gripper_base_link.STL" />
+                    <mesh filename="file://$(find inspire_description)/meshes/gripper_base_link.STL" />
                 </geometry>
             </collision>
@@ -71,5 +71,5 @@
                 <origin xyz="0 0 0" rpy="0 0 0" />
                 <geometry>
-                    <mesh filename="package://inspire_description/meshes/gripper_Link1.STL" />
+                    <mesh filename="file://$(find inspire_description)/meshes/gripper_Link1.STL" />
                 </geometry>
                 <material name="">
@@ -80,5 +80,5 @@
                 <origin xyz="0 0 0" rpy="0 0 0" />
                 <geometry>
-                    <mesh filename="package://inspire_description/meshes/gripper_Link1.STL" />
+                    <mesh filename="file://$(find inspire_description)/meshes/gripper_Link1.STL" />
                 </geometry>
             </collision>
@@ -100,5 +100,5 @@
                 <origin xyz="0 0 0" rpy="0 0 0" />
                 <geometry>
-                    <mesh filename="package://inspire_description/meshes/gripper_Link2.STL" />
+                    <mesh filename="file://$(find inspire_description)/meshes/gripper_Link2.STL" />
                 </geometry>
                 <material name="">
@@ -109,5 +109,5 @@
                 <origin xyz="0 0 0" rpy="0 0 0" />
                 <geometry>
-                    <mesh filename="package://inspire_description/meshes/gripper_Link2.STL" />
+                    <mesh filename="file://$(find inspire_description)/meshes/gripper_Link2.STL" />
                 </geometry>
             </collision>
@@ -129,5 +129,5 @@
                 <origin xyz="0 0 0" rpy="0 0 0" />
                 <geometry>
-                    <mesh filename="package://inspire_description/meshes/gripper_Link3.STL" />
+                    <mesh filename="file://$(find inspire_description)/meshes/gripper_Link3.STL" />
                 </geometry>
                 <material name="">
@@ -138,5 +138,5 @@
                 <origin xyz="0 0 0" rpy="0 0 0" />
                 <geometry>
-                    <mesh filename="package://inspire_description/meshes/gripper_Link3.STL" />
+                    <mesh filename="file://$(find inspire_description)/meshes/gripper_Link3.STL" />
                 </geometry>
             </collision>
@@ -158,5 +158,5 @@
                 <origin xyz="0 0 0" rpy="0 0 0" />
                 <geometry>
-                    <mesh filename="package://inspire_description/meshes/gripper_Link4.STL" />
+                    <mesh filename="file://$(find inspire_description)/meshes/gripper_Link4.STL" />
                 </geometry>
                 <material name="">
@@ -167,5 +167,5 @@
                 <origin xyz="0 0 0" rpy="0 0 0" />
                 <geometry>
-                    <mesh filename="package://inspire_description/meshes/gripper_Link4.STL" />
+                    <mesh filename="file://$(find inspire_description)/meshes/gripper_Link4.STL" />
                 </geometry>
             </collision>

Commit message: fix gripper

File: inspire_description/urdf/inspire_gripper.urdf.xacro (robot description, xacro)
@@ -84,10 +84,8 @@
             </collision>
         </link>
-        <joint name="gripper_joint1" type="revolute">
+        <joint name="gripper_joint1" type="fixed">
             <origin xyz="0 -0.04 0.09" rpy="0.8663 0 0" />
             <parent link="gripper_base_link" />
             <child link="gripper_Link1" />
-            <axis xyz="1 0 0" />
-            <limit lower="${joint_lower_bound}" upper="${joint_upper_bound}" effort="100" velocity="1" />
         </joint>
         <link name="gripper_Link2">
@@ -113,10 +111,8 @@
             </collision>
         </link>
-        <joint name="gripper_joint2" type="revolute">
+        <joint name="gripper_joint2" type="fixed">
             <origin xyz="0 0.022341 0.035565" rpy="-0.8663 0 0" />
             <parent link="gripper_Link1" />
             <child link="gripper_Link2" />
-            <axis xyz="-1 0 0" />
-            <limit lower="${joint_lower_bound}" upper="${joint_upper_bound}" effort="100" velocity="1" />
         </joint>
         <link name="gripper_Link3">
@@ -142,10 +138,8 @@
             </collision>
         </link>
-        <joint name="gripper_joint3" type="revolute">
+        <joint name="gripper_joint3" type="fixed">
             <origin xyz="0 0.04 0.09" rpy="-0.8663 0 0" />
             <parent link="gripper_base_link" />
             <child link="gripper_Link3" />
-            <axis xyz="-1 0 0" />
-            <limit lower="${joint_lower_bound}" upper="${joint_upper_bound}" effort="100" velocity="1" />
         </joint>
         <link name="gripper_Link4">
@@ -171,10 +165,8 @@
             </collision>
         </link>
-        <joint name="gripper_joint4" type="revolute">
+        <joint name="gripper_joint4" type="fixed">
             <origin xyz="0 -0.022341 0.035565" rpy="0.8663 0 0" />
             <parent link="gripper_Link3" />
             <child link="gripper_Link4" />
-            <axis xyz="1 0 0" />
-            <limit lower="${joint_lower_bound}" upper="${joint_upper_bound}" effort="100" velocity="1" />
         </joint>
         <!-- gripper tip virtual link -->
